File: source/smorespad.kicad_pcb (KiCad board)
At the start: 2 copper layers, 45.9 x 57.9 mm, 8 parts, among them J1 Conn_01x04, SW1 SW_Push, SW2 SW_Push, SW3 SW_Push, SW4 SW_Push, U1 XIAO_ESP32C3

Commit message: added some silkscreen, ready to order from jlc
Other:
- board text added: "emoolie"
- board text added: "s'mores pad"
Changed lines of the file:
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@@
 		(layer "Edge.Cuts")
+	)
+	(gr_text "s'mores pad"
+		(at 89.99 41.48 0)
+		(layer "F.Cu")
+		(effects
+			(font
+				(size 1.5 1.5)
+				(thickness 0.2)
+			)
+			(justify left bottom)
+		)
+	)
+	(gr_text "emoolie"
+		(at 133.89 95.85 90)
+		(layer "F.Cu")
+		(effects
+			(font
+				(size 1.5 1.5)
+				(thickness 0.2)
+			)
+			(justify left bottom)
+		)
 	)
 	(segment
